Commit message: changed urdf xacro macro name to asus_xtion

File: asus_xtion_description/urdf/asus_xtion.urdf.xacro (robot description, xacro)
@@ -11,6 +11,6 @@
 You should have received a copy of the GNU General Public License
 along with this program.  If not, see <https://www.gnu.org/licenses/>. -->
-<robot name="sensor_asus_xtion" xmlns:xacro="http://www.ros.org/wiki/xacro">
-  <xacro:macro name="sensor_asus_xtion" params="name parent *origin ">
+<robot name="asus_xtion" xmlns:xacro="http://www.ros.org/wiki/xacro">
+  <xacro:macro name="asus_xtion" params="name parent *origin ">
     <xacro:property name="M_SCALE_XTION" value="0.001"/>
     <xacro:property name="asus_xtion_pro_depth_rel_rgb_py" value="0.0270" />

Commit message: urdf file needs significant overhaul

File: asus_xtion_description/urdf/asus_xtion.urdf.xacro (robot description, xacro)
@@ -1,16 +1,13 @@
 <?xml version="1.0"?>
 <!-- Copyright (C) 2023  Miguel Ángel González Santamarta
-This program is free software: you can redistribute it and/or modify
-it under the terms of the GNU General Public License as published by
-the Free Software Foundation, either version 3 of the License, or
-(at your option) any later version.
-This program is distributed in the hope that it will be useful,
-but WITHOUT ANY WARRANTY; without even the implied warranty of
-MERCHANTABILITY or FITNESS FOR A PARTICULAR PURPOSE.  See the
-GNU General Public License for more details.
-You should have received a copy of the GNU General Public License
-along with this program.  If not, see <https://www.gnu.org/licenses/>. -->
+Copyright (C) 2024  Azmyin Md. Kamal
+BSD -3 license
+This version has only been tested for a simlulated RGB-D sensor.
+-->
 <robot name="asus_xtion" xmlns:xacro="http://www.ros.org/wiki/xacro">
-  <xacro:macro name="asus_xtion" params="name parent *origin ">
+  <xacro:macro name="asus_xtion" params="name parent_link *origin
+                                        update_rate:=30.0
+                                        image_height:=480
+                                        image_width:=640">
     <xacro:property name="M_SCALE_XTION" value="0.001"/>
     <xacro:property name="asus_xtion_pro_depth_rel_rgb_py" value="0.0270" />

Commit message: fixed  not found issue

File: asus_xtion_description/urdf/asus_xtion.urdf.xacro (robot description, xacro)
@@ -14,10 +14,20 @@
     <xacro:property name="asus_xtion_pro_cam_rel_rgb_py"   value="-0.0220" />
     <xacro:property name="M_PI" value="3.1415926535897931" />
-    <joint name="${name}_cam_rgb_joint" type="fixed">
-	  <xacro:insert_block name="origin" />
-      <parent link="${parent}"/>
-      <child link="${name}_rgb_frame" />
+    <!-- I assume Asus Xtion pro and Intel realsense camera have very similar body structures -->
+    <!-- camera body, with origin at bottom screw mount -->
+    <joint name="${name}_joint" type="fixed">
+      <xacro:insert_block name="origin" />
+      <parent link="${parent_link}"/>
+      <child link="${name}_bottom_screw_frame" />
     </joint>
-    <link name="${name}_rgb_frame">
+    <!-- Self-closing link, serves as a "fixed" reference frame for kinematic transformation -->
+    <link name="${name}_bottom_screw_frame"/>
+    <joint name="${name}_bottom_to_rgb_frame_joint" type="fixed">
+        <origin xyz="$0 0 0" rpy="0 0 0"/>
+        <parent link="${name}_bottom_screw_frame"/>
+        <child link="${name}_rgbd_frame" />
+      </joint>
+    <!-- Equivalent to ${name}_link in intel_realsense.urdf.xacro -->
+    <link name="${name}_rgbd_frame">
       <inertial>
         <mass value="0.001" />
@@ -30,5 +40,5 @@
     <joint name="${name}_rgb_optical_joint" type="fixed">
       <origin xyz="0 0 0" rpy="${-M_PI/2} 0 ${-M_PI/2}" />
-      <parent link="${name}_rgb_frame" />
+      <parent link="${name}_rgbd_frame" />
       <child link="${name}_rgb_optical_frame" />
     </joint>
@@ -45,5 +55,5 @@
       <origin xyz="0 ${asus_xtion_pro_cam_rel_rgb_py} 0"
               rpy="0 0 0"/>
-      <parent link="${name}_rgb_frame"/>
+      <parent link="${name}_rgbd_frame"/>
       <child link="${name}_cam_link"/>
     </joint>
@@ -55,10 +65,4 @@
         </geometry>
       </visual>
-      <!--collision>
-        <origin xyz="0.0 0.0 0.0" rpy="0 0 0" />
-        <geometry>
-          <box size="0.0730 .2760 0.0720"/>
-        </geometry>
-      </collision-->
       <collision>
         <origin xyz="-0.01 0.02 0.0" rpy="${-M_PI/2} -${M_PI} ${-M_PI/2}" />
@@ -77,5 +81,5 @@
     <joint name="${name}_depth_joint" type="fixed">
       <origin xyz="0 ${asus_xtion_pro_depth_rel_rgb_py} 0" rpy="0 0 0" />
-      <parent link="${name}_rgb_frame" />
+      <parent link="${name}_rgbd_frame" />
       <child link="${name}_depth_frame" />
     </joint>
@@ -106,17 +110,12 @@
     <!-- FOV and other parameters taken from original version of asus_xtion_urdf.xacro -->
     <!-- https://github.com/Juancams/kobuki_ros/blob/jazzy-devel/kobuki_description/urdf/kobuki_gazebo.urdf.xacro -->
-    <gazebo reference="${name}_depth_frame">
-      <sensor type="rgbd_camera" name="xtion_rgbd_camera">
-          <always_on>1</always_on>
-          <update_rate>30</update_rate>
-          <visualize>true</visualize>
-          <topic>rgbd_camera</topic>
-          <!-- <enable_metrics>true</enable_metrics> -->
+    <gazebo reference="${name}_rgbd_frame">
+      <sensor type="rgbd_camera" name="${name}">
           <camera>
             <horizontal_fov>1.57</horizontal_fov>
             <image>
               <format>R8G8B8</format>
-              <width>640</width>
-              <height>480</height>
+              <width>${image_width}</width>
+              <height>${image_height}</height>
             </image>
             <clip>
@@ -124,4 +123,6 @@
             <far>100</far>
           </clip>
+          <gz_frame_id>${name}_rgbd_frame</gz_frame_id>
+          <optical_frame_id>${name}_rgb_optical_frame</optical_frame_id>
           <noise>
             <type>gaussian</type>
@@ -140,4 +141,10 @@
           <!-- <gz_frame_id>${name}_depth_frame</gz_frame_id>  -->
           </camera>
+          <always_on>1</always_on>
+          <update_rate>${update_rate}</update_rate>
+          <visualize>true</visualize>
+          <gz_frame_id>${name}_rgbd_frame</gz_frame_id>
+          <topic>$(arg namespace)/sensors/${name}</topic>
+          <!-- <enable_metrics>true</enable_metrics> -->
         </sensor>
     </gazebo>

Commit message: fixed /usr/bin/bash error in urdf.xacro file

File: asus_xtion_description/urdf/asus_xtion.urdf.xacro (robot description, xacro)
@@ -24,5 +24,5 @@
     <link name="${name}_bottom_screw_frame"/>
     <joint name="${name}_bottom_to_rgb_frame_joint" type="fixed">
-        <origin xyz="$0 0 0" rpy="0 0 0"/>
+        <origin xyz="0 0 0" rpy="0 0 0"/>
         <parent link="${name}_bottom_screw_frame"/>
         <child link="${name}_rgbd_frame" />

Commit message: fixed camera image orientation problem

File: asus_xtion_description/urdf/asus_xtion.urdf.xacro (robot description, xacro)
@@ -39,5 +39,7 @@
     </link>
     <joint name="${name}_rgb_optical_joint" type="fixed">
-      <origin xyz="0 0 0" rpy="${-M_PI/2} 0 ${-M_PI/2}" />
+      <!-- <origin xyz="0 0 0" rpy="${-M_PI/2} 0 ${-M_PI/2}" /> -->
+      <!-- Gives correct image orientation -->
+      <origin xyz="0 0 0" rpy="${M_PI} 0 0" />
       <parent link="${name}_rgbd_frame" />
       <child link="${name}_rgb_optical_frame" />
@@ -93,6 +95,7 @@
       </inertial>
     </link>
+    <!-- Gives correct image orientation -->
     <joint name="${name}_cam_depth_optical_joint" type="fixed">
-      <origin xyz="0 0 0" rpy="${-M_PI/2} 0 ${-M_PI/2}" />
+      <origin xyz="0 0 0" rpy="${M_PI} 0 0" />
       <parent link="${name}_depth_frame" />
       <child link="${name}_depth_optical_frame" />
